File: hardware/current-low-cost/pcb-a/kicad/SmartBin_A.kicad_pcb (KiCad board)
At the start: 2 copper layers, 100 x 100 mm, 94 parts, among them J1 BAT_SW, J10 MCP_BUS, J11 MCP_A, J12 MCP_B, J13 OLED, J14 MPU6050, J15 RC522, J16 FLASH, J17 HC05, J18 PC_UART, J19 TB6612_CTRL, J2 BUCK_IN, J20 SERVO_SIG, J21 HC_SR04, J22 DHT, J23 DHT_LEVEL, J24 ENCODER, J25 KEYS_LID, J26 BUMPER, J27 ESTOP_2NC, J28 AO3400_ADAPTER, J29 WHITE_LED, J3 BUCK_OUT, J30 BUZZER, J31 DFPLAYER_SIG, J32 LIGHT, J33 IR_INPUTS, J4 MOTOR_PWR, J5 SERVO_PWR, J6 LOGIC_PWR, J7 EXT_REG, J8 CORE_PA, J9 CORE_PB, Q1 2N3904, Q2 2N3904, Q3 2N3904, U1 SN74AHCT125N

Commit message: Improve A1 ground stitching and add four-suite design review
Routing:
- net GND: vias 0 -> 55
